File: hardware/KiCad/watersens.sch (KiCad schematic (older format))
At the start: 72 parts, among them P1 BNC, P2 BNC, P3 BNC, P4 BNC, SW1 SW_PUSH

Commit message: short pin 7 on mux to ground.
update schematic, netlist, PCB, fills, and plots.
Connections:
- net GND: now also MUX1.7 (VEE)
- no-connect marks 38 -> 37
Changed lines of the file:
@@
 LIBS:valves
 LIBS:watersens
-LIBS:arduino_shieldsNCL
 LIBS:watersens-cache
 EELAYER 27 0
@@
 Sheet 1 1
 Title "Tentacle Shield"
-Date "22 oct 2014"
+Date "15 jul 2015"
 Rev "T1.15A"
 Comp "Whitebox Labs"
@@
 	0    1    1    0
 $EndComp
-NoConn ~ 13600 1750
 Text Notes 4550 1150 2    60   ~ 0
 PIN 1/2 : Stamp in 12C mode\nPIN 2/3 : Stamp in Serial mode
@@
 Connection ~ 14300 9400
 Connection ~ 13900 9400
+$Comp
+L GND #PWR?
+U 1 1 55A67900
+P 13750 1750
+F 0 "#PWR?" H 13750 1750 30  0001 C CNN
+F 1 "GND" H 13750 1680 30  0001 C CNN
+F 2 "" H 13750 1750 60  0000 C CNN
+F 3 "" H 13750 1750 60  0000 C CNN
+	1    13750 1750
+	0    -1   -1   0
+$EndComp
+Wire Wire Line
+	13600 1750 13750 1750
 $EndSCHEMATC

Commit message: update component lib pin labels
update labels, update to chain.
Changed lines of the file:
@@
 $EndDescr
-$Comp
-L 74HCT4052D MUX1
-U 1 1 533742EE
-P 12800 2000
-F 0 "MUX1" V 13450 2650 60  0000 C CNN
-F 1 "74HCT4052D" V 12850 2150 60  0000 C CNN
-F 2 "~" H 12800 2000 60  0000 C CNN
-F 3 "~" H 12800 2000 60  0000 C CNN
-	1    12800 2000
-	0    -1   -1   0
-$EndComp
 $Comp
 L SI8600 SIG_ISO3
@@
 $EndComp
 $Comp
-L GND #PWR27
+L GND #PWR28
 U 1 1 5337EC9B
 P 14350 9700
-F 0 "#PWR27" H 14350 9700 30  0001 C CNN
+F 0 "#PWR28" H 14350 9700 30  0001 C CNN
 F 1 "GND" H 14350 9630 30  0001 C CNN
 F 2 "" H 14350 9700 60  0000 C CNN
@@
 $EndComp
 $Comp
-L VCC #PWR26
+L VCC #PWR27
 U 1 1 5337ECBD
 P 13900 9700
-F 0 "#PWR26" H 13900 9800 30  0001 C CNN
+F 0 "#PWR27" H 13900 9800 30  0001 C CNN
 F 1 "VCC" H 13900 9800 30  0000 C CNN
 F 2 "" H 13900 9700 60  0000 C CNN
@@
 $EndComp
 $Comp
-L VCC #PWR28
+L VCC #PWR29
 U 1 1 53E8C9DA
 P 15300 1750
-F 0 "#PWR28" H 15300 1850 30  0001 C CNN
+F 0 "#PWR29" H 15300 1850 30  0001 C CNN
 F 1 "VCC" H 15300 1850 30  0000 C CNN
 F 2 "" H 15300 1750 60  0000 C CNN
@@
 Connection ~ 13900 9400
 $Comp
-L GND #PWR?
+L GND #PWR26
 U 1 1 55A67900
 P 13750 1750
-F 0 "#PWR?" H 13750 1750 30  0001 C CNN
+F 0 "#PWR26" H 13750 1750 30  0001 C CNN
 F 1 "GND" H 13750 1680 30  0001 C CNN
 F 2 "" H 13750 1750 60  0000 C CNN
@@
 Wire Wire Line
 	13600 1750 13750 1750
+$Comp
+L 74HCT4052D MUX1
+U 1 1 55A68046
+P 12800 2000
+F 0 "MUX1" V 12300 2600 60  0000 C CNN
+F 1 "74HCT4052D" V 12850 2150 60  0000 C CNN
+F 2 "~" H 12800 2000 60  0000 C CNN
+F 3 "~" H 12800 2000 60  0000 C CNN
+	1    12800 2000
+	0    -1   -1   0
+$EndComp
 $EndSCHEMATC
