File: hardware/KiCad/watersens.sch (KiCad schematic (older format))
At the start: 72 parts, among them P1 BNC, P2 BNC, P3 BNC, P4 BNC, SW1 SW_PUSH

Commit message: Update for KiCad v4
Parts:
- C1, C10, C11, C14, C15, C16, C19, C20, C4, C5, C6, C9, R1, R10, R11, R12, R13, R14, R15, R16, R18, R19, R2, R3, R4, R5, R6, R7, R8, R9: footprint ~ -> tentacle:SM0805a
- C12, C13, C17, C18, C2, C3, C7, C8, R17: footprint ~ -> tentacle:SM0805
- C21: footprint ~ -> tentacle:c_tant_X
- DCDC1, DCDC2, DCDC3, DCDC4: footprint ~ -> tentacle:R1SE_0505
- JP1, JP2, JP3, JP4, JP5, JP6, JP7, JP8, JP9: footprint ~ -> tentacle:PINHEAD1-3a
- MUX1: footprint ~ -> tentacle:SO16N
- P1, P2, P3, P4: footprint ~ -> tentacle:BNC-1337543a
- REG1, REG2, REG3, REG4: footprint ~ -> tentacle:sot89
- SHIELD1: footprint (none) -> tentacle:ARDUINO_SHIELD_040pinsa_no_outline
- SIG_ISO1, SIG_ISO2, SIG_ISO3, SIG_ISO4: footprint ~ -> tentacle:so-8a
- STP1, STP2, STP3, STP4: footprint ~ -> tentacle:Atlas_Stamp
- SW1: footprint ~ -> tentacle:B3S-1000P
